File: Kicad/rfidReader/rfidReader.kicad_pcb (KiCad board)
At the start: 2 copper layers, 33.2 x 71.5 mm, 18 parts, among them J1 USB_A, U1 WEMOS_D1_mini, U3 TPD4E05U06DQA

Commit message: kicad
Parts:
- renumbered TP1 to 3.3V, TP4 to GND, Marche2 to Marche, Validation1 to OK, TP2 to RX
Other:
- board text added: "TPD4E05U06DQA R8=R9=100 C1=4.7uf C2=100nf C3=1uf C4=100uf Diode=TVS Fuse=SS34"
Changed lines of the file:
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@@
 			(plot_on_all_layers_selection 0x00000000_00000000_00000000_00000000)
 			(disableapertmacros no)
-			(usegerberextensions no)
+			(usegerberextensions yes)
 			(usegerberattributes yes)
 			(usegerberadvancedattributes yes)
@@
 			(outputformat 1)
 			(mirror no)
-			(drillshape 1)
+			(drillshape 0)
 			(scaleselection 1)
-			(outputdirectory "")
+			(outputdirectory "../../Projet Fini/")
 		)
 	)
@@
 		(descr "LED, diameter 5.0mm, 2 pins, http://cdn-reichelt.de/documents/datenblatt/A500/LL-504BC2E-009.pdf, generated by kicad-footprint-generator")
 		(tags "LED")
-		(property "Reference" "Validation1"
+		(property "Reference" "OK"
 			(at 1.27 -3.96 0)
 			(layer "F.SilkS")
@@
 		(descr "SMD rectangular pad as test Point, square 3.0mm side length")
 		(tags "test point SMD pad rectangle square")
-		(property "Reference" "TP4"
+		(property "Reference" "GND"
 			(at 0 -2.398 0)
 			(layer "F.SilkS")
@@
 		(descr "SMD rectangular pad as test Point, square 3.0mm side length")
 		(tags "test point SMD pad rectangle square")
-		(property "Reference" "TP2"
+		(property "Reference" "RX"
 			(at 0 -2.398 0)
 			(layer "F.SilkS")
@@
 		(descr "LED, diameter 5.0mm, 2 pins, http://cdn-reichelt.de/documents/datenblatt/A500/LL-504BC2E-009.pdf, generated by kicad-footprint-generator")
 		(tags "LED")
-		(property "Reference" "Marche2"
+		(property "Reference" "Marche"
 			(at 1.27 -3.96 0)
 			(layer "F.SilkS")
@@
 		(descr "SMD rectangular pad as test Point, square 3.0mm side length")
 		(tags "test point SMD pad rectangle square")
-		(property "Reference" "TP1"
+		(property "Reference" "3.3V"
 			(at 0 -2.398 0)
 			(layer "F.SilkS")
@@
 		(layer "Edge.Cuts")
 	)
+	(gr_text "TPD4E05U06DQA\nR8=R9=100\nC1=4.7uf\nC2=100nf\nC3=1uf\nC4=100uf\nDiode=TVS\nFuse=SS34\n"
+		(at 215.65 129.7 0)
+		(layer "F.SilkS")
+		(effects
+			(font
+				(size 0.75 0.75)
+				(thickness 0.1)
+			)
+			(justify left bottom)
+		)
+	)
 	(dimension
