File: Kicad/rfidReader/rfidReader.kicad_sch (KiCad schematic)
At the start: 19 parts, among them J1 USB_A, U1 WEMOS_D1_mini, U3 TPD4E05U06DQA

Commit message: v2
Parts:
- removed Marche2: LED, LED_THT:LED_D5.0mm, symbol Device:LED
- added C5, C6, C9: 10uf, Capacitor_SMD:C_0805_2012Metric_Pad1.18x1.45mm_HandSolder, symbol Device:C
- added C7: 0.1uf, Capacitor_SMD:C_0805_2012Metric_Pad1.18x1.45mm_HandSolder, symbol Device:C
- added C8: 100nf, Capacitor_SMD:C_0805_2012Metric_Pad1.18x1.45mm_HandSolder, symbol Device:C
- added U5: AP2112K-3.3, Package_TO_SOT_SMD:SOT-23-5, symbol Regulator_Linear:AP2112K-3.3
- R9: value R -> 0.1
Connections:
- net GND: now also C5.2, C6.2, C7.2, C8.2, C9.2, U5.2 (GND)
- net VBUS: now also R9.1; no longer C3.1, C4.1, U1A1.7 (REGIN)
- net VDD renamed 3V3
- net 3V3: now also C6.1, C7.1, C8.1, C9.1, U5.5 (VOUT); no longer R9.2
- new net: C3.1, C4.1, U1A1.7 (REGIN)
- new net: C5.1, R9.2, U5.1 (VIN), U5.3 (EN)
Other:
- moved on the sheet: C3, C4, D1, F2, U1, U2, U3
